File: hardware/Body-Shield.brd (EAGLE design)
At the start: 118.1 x 53.3 mm, 77 parts

Commit message: Adding firmware, sound files, etc
Connections:
- removed net BTN12: JP9.4
- removed net CTL4: JP9.5
- removed net CTL5: JP9.6
- removed net LED12: JP8.13
- removed net N$14: JP8.12
- net BTN0: now also JP9.6; no longer JP3.6
- net BTN3: now also JP8.13; no longer JP4.8
- net LED2: now also JP9.4; no longer JP3.1
- net LED3: now also JP9.5; no longer JP4.7
- net LED5: now also JP8.12; no longer JP4.3
Routing:
- net LED5: track 34.9 -> 0.00 mm
- net LED3: track 16.5 -> 0.00 mm
- net LED2: track 15.4 -> 0.00 mm
- net BTN0: track 43.3 -> 28.7 mm
- net BTN3: track 17.8 -> 3.65 mm
Other:
- board text added: "B+"
- board text added: "B-"
- board text added: "L+"
- board text added: "L-"
Changed lines of the file:
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@@
 <layer number="47" name="Measures" color="7" fill="1" visible="no" active="yes"/>
 <layer number="48" name="Document" color="7" fill="1" visible="no" active="yes"/>
-<layer number="49" name="Reference" color="7" fill="1" visible="yes" active="yes"/>
+<layer number="49" name="Reference" color="7" fill="1" visible="no" active="yes"/>
 <layer number="50" name="dxf" color="7" fill="1" visible="no" active="yes"/>
 <layer number="51" name="tDocu" color="6" fill="1" visible="yes" active="yes"/>
@@
 <text x="-10.033" y="45.085" size="2.54" layer="21" font="vector" ratio="15" align="center">5V Only!</text>
 <text x="-13.97" y="3.81" size="1.778" layer="21" font="vector" ratio="15" align="center">Speaker</text>
+<text x="-15.24" y="17.907" size="1.27" layer="21" font="vector" ratio="15">L-</text>
+<text x="-15.24" y="19.939" size="1.27" layer="21" font="vector" ratio="15">L+</text>
+<text x="-15.24" y="21.971" size="1.27" layer="21" font="vector" ratio="15">B-</text>
+<text x="-15.24" y="24.003" size="1.27" layer="21" font="vector" ratio="15">B+</text>
 </plain>
 <attributes>
@@
 </signal>
 <signal name="LED5">
-<contactref element="JP4" pad="3"/>
 <contactref element="R18" pad="P$1"/>
-<wire x1="85.09" y1="36.83" x2="76.2" y2="45.72" width="0.254" layer="1"/>
-<wire x1="76.2" y1="45.72" x2="60.833" y2="45.72" width="0.254" layer="1"/>
-<wire x1="60.833" y1="45.72" x2="55.88" y2="50.673" width="0.254" layer="1"/>
+<contactref element="JP8" pad="12"/>
+<wire x1="85.09" y1="36.83" x2="94.107" y2="38.1" width="0" layer="19" extent="1-1"/>
 </signal>
 <signal name="LED4">
@@
 </signal>
 <signal name="LED3">
-<contactref element="JP4" pad="7"/>
 <contactref element="R9" pad="P$1"/>
-<wire x1="45.72" y1="43.2816" x2="45.72" y2="50.673" width="0.254" layer="1"/>
-<wire x1="52.0192" y1="36.9824" x2="45.72" y2="43.2816" width="0.254" layer="1"/>
-<wire x1="52.0192" y1="36.9824" x2="52.07" y2="36.83" width="0.254" layer="1"/>
+<contactref element="JP9" pad="5"/>
+<wire x1="52.07" y1="36.83" x2="91.567" y2="38.1" width="0" layer="19" extent="1-1"/>
 </signal>
 <signal name="AREF">
@@
 <contactref element="JP15" pad="4"/>
 <contactref element="R16" pad="P$2"/>
-<contactref element="JP3" pad="6"/>
 <wire x1="-9.61" y1="36.02" x2="-9.61" y2="36.11" width="0.254" layer="1"/>
 <wire x1="-9.61" y1="36.11" x2="-8.89" y2="36.83" width="0.254" layer="1"/>
@@
 <wire x1="-6.35" y1="38.1" x2="-3.81" y2="40.64" width="0.254" layer="16"/>
 <wire x1="-3.81" y1="40.64" x2="16.383" y2="40.64" width="0.254" layer="16"/>
-<wire x1="16.383" y1="40.64" x2="26.67" y2="50.927" width="0.254" layer="16"/>
+<contactref element="JP9" pad="6"/>
+<wire x1="16.383" y1="40.64" x2="91.313" y2="35.56" width="0" layer="19" extent="16-16"/>
 </signal>
 <signal name="LED0">
@@
 </signal>
 <signal name="BTN3">
-<contactref element="JP4" pad="8"/>
 <contactref element="JP16" pad="4"/>
 <contactref element="R10" pad="P$2"/>
-<wire x1="43.2816" y1="36.9824" x2="43.2816" y2="50.8" width="0.254" layer="1"/>
-<wire x1="43.2816" y1="50.8" x2="43.18" y2="50.927" width="0.254" layer="1"/>
-<wire x1="43.2816" y1="36.9824" x2="43.18" y2="36.83" width="0.254" layer="1"/>
 <wire x1="39.92" y1="36.02" x2="39.92" y2="36.11" width="0.254" layer="1"/>
 <wire x1="39.92" y1="36.11" x2="40.64" y2="36.83" width="0.254" layer="1"/>
 <wire x1="40.64" y1="36.83" x2="43.18" y2="36.83" width="0.254" layer="1"/>
+<contactref element="JP8" pad="13"/>
+<wire x1="43.18" y1="36.83" x2="93.853" y2="40.64" width="0" layer="19" extent="1-1"/>
 </signal>
 <signal name="BTN4">
@@
 </signal>
 <signal name="LED2">
-<contactref element="JP3" pad="1"/>
 <contactref element="R6" pad="P$1"/>
-<wire x1="35.56" y1="36.83" x2="35.56" y2="45.72" width="0.254" layer="1"/>
-<wire x1="35.56" y1="45.72" x2="39.37" y2="49.53" width="0.254" layer="1"/>
-<wire x1="39.37" y1="49.53" x2="39.37" y2="50.673" width="0.254" layer="1"/>
+<contactref element="JP9" pad="4"/>
+<wire x1="35.56" y1="36.83" x2="91.313" y2="40.64" width="0" layer="19" extent="1-1"/>
 </signal>
 <signal name="SIG-">
@@
 <wire x1="82.55" y1="40.64" x2="85.09" y2="43.18" width="0.254" layer="16"/>
 <wire x1="85.09" y1="43.18" x2="91.567" y2="43.18" width="0.254" layer="16"/>
-</signal>
-<signal name="BTN12">
-<contactref element="JP9" pad="4"/>
-</signal>
-<signal name="CTL4">
-<contactref element="JP9" pad="5"/>
-</signal>
-<signal name="CTL5">
-<contactref element="JP9" pad="6"/>
 </signal>
 <signal name="A13">
@@
 <wire x1="89.8652" y1="52.07" x2="90.0176" y2="52.2224" width="0.254" layer="1"/>
 </signal>
-<signal name="LED12">
-<contactref element="JP8" pad="13"/>
-</signal>
-<signal name="N$14">
-<contactref element="JP8" pad="12"/>
-</signal>
 <signal name="N$15">
